File: reviung34/pcb/reviung34.kicad_pcb (KiCad board)
At the start: 2 copper layers, 214.3 x 107.1 mm, 95 parts, among them SW1 SW_PUSH, SW10 SW_PUSH, SW11 SW_PUSH, SW12 SW_PUSH, SW13 SW_PUSH, SW14 SW_PUSH, SW15 SW_PUSH, SW16 SW_PUSH, SW17 SW_PUSH, SW18 SW_PUSH, SW19 SW_PUSH, SW2 SW_PUSH, SW20 SW_PUSH, SW21 SW_PUSH, SW22 SW_PUSH, SW23 SW_PUSH, SW24 SW_PUSH, SW25 SW_PUSH, SW26 SW_PUSH, SW27 SW_PUSH, SW28 SW_PUSH, SW29 SW_PUSH, SW3 SW_PUSH, SW30 SW_PUSH, SW31 SW_PUSH, SW32 SW_PUSH, SW33 SW_PUSH, SW34 SW_PUSH, SW35 SW_PUSH, SW4 SW_PUSH, SW5 SW_PUSH, SW6 SW_PUSH, SW7 SW_PUSH, SW8 SW_PUSH, SW9 SW_PUSH, U1 ProMicro

Commit message: reviung34: hotswap
Parts:
- D1: footprint _reviung-kbd:D3_SMD_1side -> Button_Switch_SMD:SW_SPST_B3SL-1002P
- D10, D11, D12, D13, D14, D15, D16, D17, D18, D19, D2, D20, D21, D22, D23, D24, D25, D26, D27, D28, D29, D3, D30, D31, D32, D33, D34, D4, D5, D6, D7, D8, D9: footprint _reviung-kbd:D3_SMD_1side -> ScottoKeebs_Components:Diode_SOD-123
- RESET1: footprint _reviung-kbd:ResetSW_1side -> kbd:ResetSW_1side
- RGB1, RGB2, RGB3, RGB4, RGB5, RGB6, RGB7, RGB8, RGB9: footprint _reviung-kbd:LED_WS2812B_PLCC4_5.0x5.0mm_P3.2mm -> ScottoKeebs_Components:LED_WS2812B
- SW1, SW10, SW11, SW12, SW13, SW14, SW15, SW16, SW19, SW2, SW20, SW21, SW22, SW23, SW24, SW25, SW26, SW27, SW28, SW29, SW3, SW30, SW31, SW32, SW33, SW34, SW4, SW5, SW6, SW7, SW8, SW9: footprint _reviung-kbd:MXOnly-1U-NoLED -> ScottoKeebs_Hotswap:Hotswap_MX_1.00u
- SW17: footprint _reviung-kbd:MXOnly-1U-5pinRcut -> ScottoKeebs_Hotswap:Hotswap_MX_1.00u
- SW18: footprint _reviung-kbd:MXOnly-1U-5pinLcut -> ScottoKeebs_Hotswap:Hotswap_MX_1.00u
- SW35: footprint _reviung-kbd:MXOnly-2U-NoLED-or1Ux2 -> ScottoKeebs_Hotswap:Hotswap_MX_1.00u
- U1: footprint _reviung-kbd:ProMicro -> ScottoKeebs_MCU:Arduino_Pro_Micro
Connections:
- RGB9 pad 2: Net-(RGB9-Pad2) -> unconnected-(RGB9-DOUT-Pad2)
- U1 pad 12: Net-(U1-Pad12) -> unconnected-(U1-9/B5-Pad12)
- U1 pad 2: Net-(U1-Pad2) -> unconnected-(U1-RX1/D2-Pad2)
- U1 pad 24: Net-(U1-Pad24) -> unconnected-(U1-RAW-Pad24)
- U1 pad 5: Net-(U1-Pad5) -> unconnected-(U1-2/D1/SDA-Pad5)
- U1 pad 6: Net-(U1-Pad6) -> unconnected-(U1-3/D0/SCL-Pad6)
Routing:
- net col7: track 115.7 -> 260.8 mm, vias 0 -> 1
- net col4: track 145.1 -> 0.00 mm
- net col5: track 132.5 -> 0.00 mm
- net col2: track 161.1 -> 293.5 mm
- net col0: track 147.2 -> 40.2 mm, vias 1 -> 0
- net row2: track 342.4 -> 449.3 mm, vias 2 -> 3
- net col1: track 140.3 -> 40.2 mm, vias 1 -> 0
- net row3: track 322.8 -> 422.9 mm, vias 3 -> 4
- net (no net): track 0.00 -> 59.2 mm
- net reset: track 50.4 -> 0.00 mm
- net GND: track 103.7 -> 154.1 mm, vias 47 -> 46
- net Net-(RGB1-DOUT): track 36.0 -> 0.00 mm
- net col6: track 133.5 -> 169.4 mm, vias 1 -> 2
- net col3: track 147.3 -> 111.4 mm, vias 2 -> 1
- net Net-(D18-A): track 38.5 -> 15.3 mm
Other:
- net class Default removed
