File: reviung34/pcb-top-plate/pcb-top-plate-rev1.kicad_pcb (KiCad board)
At the start: 2 copper layers, 214.3 x 101.2 mm, 42 parts

Commit message: reviung34: hotswap
Other:
- net class Default removed
