File: reviung5/pcb/ver1.0/reviung5.kicad_pcb (KiCad board)
At the start: 2 copper layers, 99.7 x 51 mm, 26 parts, among them SW1 SW_PUSH, SW2 SW_PUSH, SW3 SW_PUSH, SW4 SW_PUSH, SW5 SW_PUSH, U1 ProMicro

Commit message: reviung5: two encoders
Connections:
- RESW2 pad A: padA -> padC
- RESW2 pad B: padB -> padD
- RGB4 pad 2: Net-(RGB4-Pad2) -> unconnected-(RGB4-DOUT-Pad2)
- U1 pad 12: Net-(U1-Pad12) -> unconnected-(U1-9/B5-Pad12)
- U1 pad 13: Net-(U1-Pad13) -> unconnected-(U1-B6/10-Pad13)
- U1 pad 14: Net-(U1-Pad14) -> unconnected-(U1-B2/16-Pad14)
- U1 pad 15: Net-(U1-Pad15) -> unconnected-(U1-B3/14-Pad15)
- U1 pad 16: Net-(U1-Pad16) -> unconnected-(U1-B1/15-Pad16)
- U1 pad 17: Net-(U1-Pad17) -> unconnected-(U1-F7/A0-Pad17)
- U1 pad 18: Net-(U1-Pad18) -> padC
- U1 pad 19: Net-(U1-Pad19) -> padD
- U1 pad 2: Net-(U1-Pad2) -> unconnected-(U1-RX1/D2-Pad2)
- U1 pad 24: Net-(U1-Pad24) -> unconnected-(U1-RAW-Pad24)
Routing:
- net padB: track 120.6 -> 57.0 mm
- net padD: track 0.00 -> 58.9 mm
- net padC: track 0.00 -> 56.0 mm
- net padA: track 116.4 -> 61.9 mm
Other:
- net class Default removed
